File: keyboard.kicad_sch (KiCad schematic)
At the start: 208 parts, among them J2 USB_C_Receptacle_USB2.0_16P, J3 Conn_01x04, J4 Conn_01x05, SW1 SW_Push, SW2 SW_Push, U1 RP2040, U2 NCP1117-3.3_SOT223, U3 W25Q128JVS, U4 SRV05-4, Y1 Crystal_GND24

Commit message: HS to regular switch footprint, component layout possibly complete
Parts:
- removed MX1, MX10, MX11, MX12, MX13, MX14, MX15, MX16, MX17, MX18, MX19, MX2, MX20, MX21, MX22, MX23, MX24, MX25, MX26, MX27, MX28, MX29, MX3, MX30, MX31, MX33, MX34, MX35, MX36, MX37, MX38, MX39, MX4, MX40, MX41, MX42, MX43, MX44, MX46, MX48, MX49, MX5, MX50, MX51, MX52, MX53, MX54, MX55, MX56, MX57, MX58, MX59, MX6, MX60, MX61, MX62, MX63, MX64, MX65, MX66, MX67, MX68, MX69, MX7, MX70, MX71, MX73, MX74, MX78, MX79, MX8, MX80, MX81, MX82, MX83, MX84, MX9: MX_SW_HS, PCM_marbastlib-mx:SW_MX_HS_CPG151101S11_1u, symbol PCM_marbastlib-mx:MX_SW_HS_CPG151101S11
- removed MX32, MX45: MX_SW_HS, PCM_marbastlib-mx:SW_MX_HS_CPG151101S11_1.5u, symbol PCM_marbastlib-mx:MX_SW_HS_CPG151101S11
- removed MX47, MX72: MX_SW_HS, PCM_marbastlib-mx:SW_MX_HS_CPG151101S11_1.75u, symbol PCM_marbastlib-mx:MX_SW_HS_CPG151101S11
- removed MX75, MX76, MX77: MX_SW_HS, PCM_marbastlib-mx:SW_MX_HS_CPG151101S11_1.25u, symbol PCM_marbastlib-mx:MX_SW_HS_CPG151101S11
- removed U2: NCP1117-3.3_SOT223, Package_TO_SOT_SMD:SOT-223-3_TabPin2, symbol Regulator_Linear:NCP1117-3.3_SOT223
- added MX1, MX10, MX11, MX12, MX13, MX14, MX15, MX16, MX17, MX18, MX19, MX2, MX20, MX21, MX22, MX23, MX24, MX25, MX26, MX27, MX28, MX29, MX3, MX30, MX31, MX33, MX34, MX35, MX36, MX37, MX38, MX39, MX4, MX40, MX41, MX42, MX43, MX44, MX46, MX48, MX49, MX5, MX50, MX51, MX52, MX53, MX54, MX55, MX56, MX57, MX58, MX59, MX6, MX60, MX61, MX62, MX63, MX64, MX65, MX66, MX67, MX68, MX69, MX7, MX70, MX71, MX73, MX74, MX78, MX79, MX8, MX80, MX81, MX82, MX83, MX84, MX9: MX_SW_solder, PCM_marbastlib-mx:SW_MX_1u, symbol PCM_marbastlib-mx:MX_SW_solder
- added MX32, MX45: MX_SW_solder, PCM_marbastlib-mx:SW_MX_1.5u, symbol PCM_marbastlib-mx:MX_SW_solder
- added MX47, MX72: MX_SW_solder, PCM_marbastlib-mx:SW_MX_1.75u, symbol PCM_marbastlib-mx:MX_SW_solder
- added MX75, MX76, MX77: MX_SW_solder, PCM_marbastlib-mx:SW_MX_1.25u, symbol PCM_marbastlib-mx:MX_SW_solder
- added U2: XC6206PxxxMR, Package_TO_SOT_SMD:SOT-23-3, symbol Regulator_Linear:XC6206PxxxMR
Connections:
- net +3V3: now also U2.2 (VO)
- net +5V: now also U2.3 (VI)
- net COL0: now also MX1.1, MX15.1, MX29.1, MX43.1, MX57.1, MX71.1
- net COL1: now also MX16.1, MX2.1, MX30.1, MX44.1, MX58.1, MX72.1
- net COL10: now also MX11.1, MX25.1, MX39.1, MX53.1, MX67.1, MX81.1
- net COL11: now also MX12.1, MX26.1, MX40.1, MX54.1, MX68.1, MX82.1
- net COL12: now also MX13.1, MX27.1, MX41.1, MX55.1, MX69.1, MX83.1
- net COL13: now also MX14.1, MX28.1, MX42.1, MX56.1, MX70.1, MX84.1
- net COL2: now also MX17.1, MX3.1, MX31.1, MX45.1, MX59.1, MX73.1
- net COL3: now also MX18.1, MX32.1, MX4.1, MX46.1, MX60.1, MX74.1
- net COL4: now also MX19.1, MX33.1, MX47.1, MX5.1, MX61.1, MX75.1
- net COL5: now also MX20.1, MX34.1, MX48.1, MX6.1, MX62.1, MX76.1
- net COL6: now also MX21.1, MX35.1, MX49.1, MX63.1, MX7.1, MX77.1
- net COL7: now also MX22.1, MX36.1, MX50.1, MX64.1, MX78.1, MX8.1
- net COL8: now also MX23.1, MX37.1, MX51.1, MX65.1, MX79.1, MX9.1
- net COL9: now also MX10.1, MX24.1, MX38.1, MX52.1, MX66.1, MX80.1
- net GND: now also U2.1 (GND)
- net at D81.2 (A): now also MX81.2
- net at D70.2 (A): now also MX70.2
- net at D9.2 (A): now also MX9.2
- net at D80.2 (A): now also MX80.2
- net at D71.2 (A): now also MX71.2
- net at D21.2 (A): now also MX21.2
- net at D63.2 (A): now also MX63.2
- net at D56.2 (A): now also MX56.2
- net at D83.2 (A): now also MX83.2
- net at D65.2 (A): now also MX65.2
- net at D55.2 (A): now also MX55.2
- net at D72.2 (A): now also MX72.2
- net at D40.2 (A): now also MX40.2
- net at D49.2 (A): now also MX49.2
- net at D12.2 (A): now also MX12.2
- net at D52.2 (A): now also MX52.2
- net at D27.2 (A): now also MX27.2
- net at D74.2 (A): now also MX74.2
- net at D29.2 (A): now also MX29.2
- net at D24.2 (A): now also MX24.2
- net at D42.2 (A): now also MX42.2
- net at D76.2 (A): now also MX76.2
- net at D26.2 (A): now also MX26.2
- net at D45.2 (A): now also MX45.2
- net at D35.2 (A): now also MX35.2
- net at D37.2 (A): now also MX37.2
- net at D84.2 (A): now also MX84.2
- net at D4.2 (A): now also MX4.2
- net at D13.2 (A): now also MX13.2
- net at D32.2 (A): now also MX32.2
- net at D8.2 (A): now also MX8.2
- net at D19.2 (A): now also MX19.2
- net at D69.2 (A): now also MX69.2
- net at D73.2 (A): now also MX73.2
- net at D58.2 (A): now also MX58.2
- net at D62.2 (A): now also MX62.2
- net at D15.2 (A): now also MX15.2
- net at D6.2 (A): now also MX6.2
- net at D34.2 (A): now also MX34.2
- net at D59.2 (A): now also MX59.2
- net at D82.2 (A): now also MX82.2
- net at D3.2 (A): now also MX3.2
- net at D14.2 (A): now also MX14.2
- net at D18.2 (A): now also MX18.2
- net at D66.2 (A): now also MX66.2
- net at D38.2 (A): now also MX38.2
- net at D51.2 (A): now also MX51.2
- net at D36.2 (A): now also MX36.2
- net at D28.2 (A): now also MX28.2
- net at D30.2 (A): now also MX30.2
- net at D61.2 (A): now also MX61.2
- net at D2.2 (A): now also MX2.2
- net at D7.2 (A): now also MX7.2
- net at D11.2 (A): now also MX11.2
- net at D31.2 (A): now also MX31.2
- net at D79.2 (A): now also MX79.2
- net at D64.2 (A): now also MX64.2
- net at D5.2 (A): now also MX5.2
- net at D53.2 (A): now also MX53.2
- net at D1.2 (A): now also MX1.2
- net at D75.2 (A): now also MX75.2
- net at D47.2 (A): now also MX47.2
- net at D41.2 (A): now also MX41.2
- net at D25.2 (A): now also MX25.2
- net at D10.2 (A): now also MX10.2
- net at D44.2 (A): now also MX44.2
- net at D46.2 (A): now also MX46.2
- net at D67.2 (A): now also MX67.2
- net at D23.2 (A): now also MX23.2
- net at D33.2 (A): now also MX33.2
- net at D48.2 (A): now also MX48.2
- net at D77.2 (A): now also MX77.2
- net at D22.2 (A): now also MX22.2
- net at D43.2 (A): now also MX43.2
- net at D17.2 (A): now also MX17.2
- net at D16.2 (A): now also MX16.2
- net at D54.2 (A): now also MX54.2
- net at D60.2 (A): now also MX60.2
- net at D57.2 (A): now also MX57.2
- net at D78.2 (A): now also MX78.2
- net at D68.2 (A): now also MX68.2
- net at D39.2 (A): now also MX39.2
- net at D50.2 (A): now also MX50.2
- net at D20.2 (A): now also MX20.2

Commit message: component layout complete, remove 4-pin connector
Parts:
- removed J3: Conn_01x04, Connector_JST:JST_SH_SM04B-SRSS-TB_1x04-1MP_P1.00mm_Horizontal, symbol Connector_Generic:Conn_01x04
- removed U4: SRV05-4, Package_TO_SOT_SMD:SOT-23-6, symbol Power_Protection:SRV05-4
- added D85: PRTR5V0U2X, Package_TO_SOT_SMD:SOT-143, symbol Power_Protection:PRTR5V0U2X
- MX1: value MX_SW_solder -> ESC
- MX10: value MX_SW_solder -> F9
- MX11: value MX_SW_solder -> F10
- MX12: value MX_SW_solder -> F11
- MX13: value MX_SW_solder -> F12
- MX14: value MX_SW_solder -> PrtSc/NmLk
- MX15: value MX_SW_solder -> Pause/ScrLk
- MX16: value MX_SW_solder -> Delete/Insert
- MX17: value MX_SW_solder -> ~'
- MX18: value MX_SW_solder -> !1
- MX19: value MX_SW_solder -> @2
- MX2: value MX_SW_solder -> F1
- MX20: value MX_SW_solder -> #3
- MX21: value MX_SW_solder -> $4
- MX22: value MX_SW_solder -> %5
- MX23: value MX_SW_solder -> ^6
- MX24: value MX_SW_solder -> &7
- MX25: value MX_SW_solder -> *8
- MX26: value MX_SW_solder -> (9
- MX27: value MX_SW_solder -> )0
- MX28: value MX_SW_solder -> _-
- MX29: value MX_SW_solder -> +=
- MX3: value MX_SW_solder -> F2
- MX30: value MX_SW_solder -> Backspace
- MX31: value MX_SW_solder -> Home
- MX32: value MX_SW_solder -> Tab
- MX33: value MX_SW_solder -> Q
- MX34: value MX_SW_solder -> W
- MX35: value MX_SW_solder -> E
- MX36: value MX_SW_solder -> R
- MX37: value MX_SW_solder -> T
- MX38: value MX_SW_solder -> Y
- MX39: value MX_SW_solder -> U
- MX4: value MX_SW_solder -> F3
- MX40: value MX_SW_solder -> I
- MX41: value MX_SW_solder -> O
- MX42: value MX_SW_solder -> P
- MX43: value MX_SW_solder -> {[
- MX44: value MX_SW_solder -> }]
- MX45: value MX_SW_solder -> |\
- MX46: value MX_SW_solder -> PageUp
- MX47: value MX_SW_solder -> CapsLock
- MX48: value MX_SW_solder -> A
- MX49: value MX_SW_solder -> S
- MX5: value MX_SW_solder -> F4
- MX50: value MX_SW_solder -> D
- MX51: value MX_SW_solder -> F
- MX52: value MX_SW_solder -> G
- MX53: value MX_SW_solder -> H
- MX54: value MX_SW_solder -> J
- MX55: value MX_SW_solder -> K
- MX56: value MX_SW_solder -> L
- MX57: value MX_SW_solder -> :;
- MX58: value MX_SW_solder -> "'
- MX59: value MX_SW_solder -> Enter
- MX6: value MX_SW_solder -> F5
- MX60: value MX_SW_solder -> PageDown
- MX61, MX72: value MX_SW_solder -> Shift
- MX62: value MX_SW_solder -> Z
- MX63: value MX_SW_solder -> X
- MX64: value MX_SW_solder -> C
- MX65: value MX_SW_solder -> V
- MX66: value MX_SW_solder -> B
- MX67: value MX_SW_solder -> N
- MX68: value MX_SW_solder -> M
- MX69: value MX_SW_solder -> <,
- MX7: value MX_SW_solder -> F6
- MX70: value MX_SW_solder -> >.
- MX71: value MX_SW_solder -> ?/
- MX73: value MX_SW_solder -> UpArrow
- MX74: value MX_SW_solder -> End
- MX75, MX81: value MX_SW_solder -> Ctrl
- MX76: value MX_SW_solder -> Win
- MX77, MX79: value MX_SW_solder -> Alt
- MX78: value MX_SW_solder -> S[acebar
- MX8: value MX_SW_solder -> F7
- MX80: value MX_SW_solder -> Fn
- MX82: value MX_SW_solder -> LeftArrow
- MX83: value MX_SW_solder -> DownArrow
- MX84: value MX_SW_solder -> RightArrow
- MX9: value MX_SW_solder -> F8
Connections:
- net +5V: now also D85.4 (VCC)
- net COL0: now also MX17.1, MX32.1, MX47.1, MX61.1, MX75.1, U1.32 (GPIO21); no longer MX15.1, MX29.1, MX43.1, MX57.1, MX71.1, U1.2 (GPIO0)
- net COL1: now also MX18.1, MX33.1, MX48.1, MX62.1, MX76.1, U1.34 (GPIO22); no longer MX16.1, MX30.1, MX44.1, MX58.1, MX72.1, U1.3 (GPIO1)
- net COL10: now also MX27.1, MX42.1, MX57.1, MX71.1, U1.8 (GPIO6); no longer MX25.1, MX39.1, MX53.1, MX67.1, U1.13 (GPIO10)
- net COL11: now also MX13.1, MX28.1, MX43.1, MX58.1, MX72.1, U1.11 (GPIO8); no longer MX26.1, MX40.1, MX54.1, MX68.1, U1.14 (GPIO11)
- net COL12: now also MX14.1, MX29.1, MX44.1, U1.9 (GPIO7); no longer MX13.1, MX27.1, MX41.1, MX55.1, MX69.1, MX83.1, U1.15 (GPIO12)
- net COL13: now also MX15.1, MX30.1, MX45.1, MX59.1, MX73.1, MX83.1, U1.13 (GPIO10); no longer MX14.1, MX28.1, MX42.1, MX56.1, MX70.1, MX84.1, U1.16 (GPIO13)
- net COL2: now also MX19.1, MX34.1, MX49.1, MX63.1, MX77.1, U1.35 (GPIO23); no longer MX17.1, MX31.1, MX45.1, MX59.1, MX73.1, U1.4 (GPIO2)
- net COL3: now also MX20.1, MX35.1, MX50.1, MX64.1, U1.36 (GPIO24); no longer MX18.1, MX32.1, MX46.1, MX60.1, MX74.1, U1.5 (GPIO3)
- net COL4: now also MX21.1, MX36.1, MX51.1, MX65.1, U1.37 (GPIO25); no longer MX19.1, MX33.1, MX47.1, MX61.1, MX75.1, U1.6 (GPIO4)
- net COL5: now also MX22.1, MX37.1, MX52.1, MX66.1, MX78.1, U1.38 (GPIO26/ADC0); no longer MX20.1, MX34.1, MX48.1, MX62.1, MX76.1, U1.7 (GPIO5)
- net COL6: now also MX23.1, MX38.1, MX53.1, MX67.1, U1.39 (GPIO27/ADC1); no longer MX21.1, MX35.1, MX49.1, MX63.1, MX77.1, U1.8 (GPIO6)
- net COL7: now also MX24.1, MX39.1, MX54.1, MX68.1, U1.6 (GPIO4); no longer MX22.1, MX36.1, MX50.1, MX64.1, MX78.1, U1.9 (GPIO7)
- net COL8: now also MX25.1, MX40.1, MX55.1, MX69.1, U1.7 (GPIO5); no longer MX23.1, MX37.1, MX51.1, MX65.1, U1.11 (GPIO8)
- net COL9: now also MX26.1, MX41.1, MX56.1, MX70.1; no longer MX24.1, MX38.1, MX52.1, MX66.1
- net GND: now also D85.1 (GND)
- net ROW0: now also D15.1 (K), D16.1 (K), U1.2 (GPIO0); no longer U1.17 (GPIO14)
- net ROW1: now also D29.1 (K), D30.1 (K), D31.1 (K), U1.3 (GPIO1); no longer D15.1 (K), D16.1 (K), U1.18 (GPIO15)
- net ROW2: now also D43.1 (K), D44.1 (K), D45.1 (K), D46.1 (K), U1.4 (GPIO2); no longer D29.1 (K), D30.1 (K), D31.1 (K), U1.27 (GPIO16)
- net ROW3: now also D57.1 (K), D58.1 (K), D59.1 (K), D60.1 (K), U1.41 (GPIO29/ADC3); no longer D43.1 (K), D44.1 (K), D45.1 (K), D46.1 (K), U1.28 (GPIO17)
- net ROW4: now also D71.1 (K), D72.1 (K), D73.1 (K), D74.1 (K), U1.40 (GPIO28/ADC2); no longer D57.1 (K), D58.1 (K), D59.1 (K), D60.1 (K), U1.29 (GPIO18)
- net ROW5: now also U1.31 (GPIO20); no longer D71.1 (K), D72.1 (K), D73.1 (K), D74.1 (K), U1.30 (GPIO19)
- net USB_D+: now also D85.3 (I/O2)
- net USB_D-: now also D85.2 (I/O1)
- new net COL14: MX16.1, MX31.1, MX46.1, MX60.1, MX74.1, MX84.1, U1.14 (GPIO11)
- no-connect marks 14 -> 11
Other:
- moved on the sheet: D15, D16, D17, D18, D19, D20, D21, D22, D23, D24, D25, D26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
