File: leds.kicad_sch (KiCad schematic)
At the start: 84 parts

Commit message: add logic level shifter to top sheet
Parts:
- renumbered LED30 to LED29, LED31 to LED30, LED32 to LED31, LED29 to LED32, LED45 to LED44, LED46 to LED45, LED47 to LED46, LED44 to LED47, LED60 to LED59, LED61 to LED60, LED59 to LED61, LED80 to LED78, LED83 to LED79, LED84 to LED80, LED85 to LED81, LED86 to LED82, LED87 to LED83, LED88 to LED84
Connections:
- net +5V: now also LED39.3 (VDD), LED40.3 (VDD), LED41.3 (VDD), LED42.3 (VDD), LED43.3 (VDD), LED44.3 (VDD), LED45.3 (VDD), LED46.3 (VDD), LED47.3 (VDD), LED48.3 (VDD), LED49.3 (VDD), LED50.3 (VDD), LED51.3 (VDD), LED52.3 (VDD), LED53.3 (VDD), LED54.3 (VDD), LED55.3 (VDD), LED56.3 (VDD), LED57.3 (VDD), LED58.3 (VDD), LED59.3 (VDD), LED60.3 (VDD), LED61.1 (VSS), LED62.1 (VSS), LED63.1 (VSS), LED64.1 (VSS), LED65.1 (VSS), LED66.1 (VSS), LED67.1 (VSS), LED68.1 (VSS), LED69.1 (VSS), LED70.1 (VSS), LED71.1 (VSS), LED72.1 (VSS), LED73.1 (VSS), LED74.1 (VSS), LED75.3 (VDD), LED76.3 (VDD), LED77.3 (VDD), LED78.3 (VDD), LED79.3 (VDD), LED80.3 (VDD), LED81.3 (VDD), LED82.3 (VDD), LED83.3 (VDD), LED84.3 (VDD)
- net GND: now also LED33.1 (VSS), LED34.1 (VSS), LED35.1 (VSS), LED36.1 (VSS), LED37.1 (VSS), LED38.1 (VSS), LED39.1 (VSS), LED40.1 (VSS), LED41.1 (VSS), LED42.1 (VSS), LED43.1 (VSS), LED44.1 (VSS), LED45.1 (VSS), LED46.1 (VSS), LED47.1 (VSS), LED48.1 (VSS), LED49.1 (VSS), LED50.1 (VSS), LED51.1 (VSS), LED52.1 (VSS), LED53.1 (VSS), LED54.1 (VSS), LED55.1 (VSS), LED56.1 (VSS), LED57.1 (VSS), LED58.1 (VSS), LED59.1 (VSS), LED60.1 (VSS), LED61.3 (VDD), LED62.3 (VDD), LED63.3 (VDD), LED64.3 (VDD), LED65.3 (VDD), LED66.3 (VDD), LED67.3 (VDD), LED68.3 (VDD), LED69.3 (VDD), LED70.3 (VDD), LED71.3 (VDD), LED72.3 (VDD), LED73.3 (VDD), LED74.3 (VDD), LED75.1 (VSS), LED76.1 (VSS), LED77.1 (VSS), LED78.1 (VSS), LED79.1 (VSS), LED80.1 (VSS), LED81.1 (VSS), LED82.1 (VSS), LED83.1 (VSS), LED84.1 (VSS)
- net at LED83.2 (DIN): now also LED84.4 (DOUT)
- net at LED83.4 (DOUT): now also LED82.2 (DIN)
- net at LED81.2 (DIN): now also LED82.4 (DOUT)
- net at LED81.4 (DOUT): now also LED80.2 (DIN)
- net at LED69.2 (DIN): now also LED70.4 (DOUT)
- net at LED69.4 (DOUT): now also LED68.2 (DIN)
- net at LED80.4 (DOUT): now also LED79.2 (DIN)
- net at LED65.2 (DIN): now also LED66.4 (DOUT)
- net at LED65.4 (DOUT): now also LED64.2 (DIN)
- net at LED70.2 (DIN): now also LED71.4 (DOUT)
- net at LED75.2 (DIN): now also LED76.4 (DOUT)
- net at LED46.2 (DIN): now also LED45.4 (DOUT)
- net at LED46.4 (DOUT): now also LED60.2 (DIN)
- net at LED72.2 (DIN): now also LED73.4 (DOUT)
- net at LED72.4 (DOUT): now also LED71.2 (DIN)
- net at LED34.2 (DIN): now also LED33.4 (DOUT)
- net at LED34.4 (DOUT): now also LED35.2 (DIN)
- net at LED79.4 (DOUT): now also LED78.2 (DIN)
- net at LED68.4 (DOUT): now also LED67.2 (DIN)
- net at LED74.2 (DIN): now also LED84.2 (DIN)
- net at LED74.4 (DOUT): now also LED73.2 (DIN)
- net at LED38.2 (DIN): now also LED37.4 (DOUT)
- net at LED38.4 (DOUT): now also LED39.2 (DIN)
- net at LED57.2 (DIN): now also LED58.4 (DOUT)
- net at LED57.4 (DOUT): now also LED56.2 (DIN)
- net at LED61.2 (DIN): now also LED62.4 (DOUT)
- net at LED61.4 (DOUT): now also LED47.4 (DOUT)
- net at LED77.2 (DIN): now also LED78.4 (DOUT)
- net at LED77.4 (DOUT): now also LED76.2 (DIN)
- net at LED58.2 (DIN): now also LED59.4 (DOUT)
- net at LED32.4 (DOUT): now also LED33.2 (DIN)
- net at LED63.2 (DIN): now also LED64.4 (DOUT)
- net at LED63.4 (DOUT): now also LED62.2 (DIN)
- net at LED39.4 (DOUT): now also LED40.2 (DIN)
- net at LED67.4 (DOUT): now also LED66.2 (DIN)
- net at LED44.2 (DIN): now also LED43.4 (DOUT)
- net at LED44.4 (DOUT): now also LED45.2 (DIN)
- net at LED50.2 (DIN): now also LED51.4 (DOUT)
- net at LED50.4 (DOUT): now also LED49.2 (DIN)
- net at LED56.4 (DOUT): now also LED55.2 (DIN)
- net at LED48.2 (DIN): now also LED49.4 (DOUT)
- net at LED48.4 (DOUT): now also LED47.2 (DIN)
- net at LED55.4 (DOUT): now also LED54.2 (DIN)
- net at LED42.2 (DIN): now also LED41.4 (DOUT)
- net at LED42.4 (DOUT): now also LED43.2 (DIN)
- net at LED51.2 (DIN): now also LED52.4 (DOUT)
- net at LED53.2 (DIN): now also LED54.4 (DOUT)
- net at LED53.4 (DOUT): now also LED52.2 (DIN)
- net at LED59.2 (DIN): now also LED60.4 (DOUT)
- net at LED36.2 (DIN): now also LED35.4 (DOUT)
- net at LED36.4 (DOUT): now also LED37.2 (DIN)
- net at LED41.2 (DIN): now also LED40.4 (DOUT)
Other:
- moved on the sheet: LED1, LED10, LED11, LED12, LED13, LED14, LED15, LED16, LED17, LED18, LED19, LED2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
