File: keyboard.kicad_pcb (KiCad board)
At the start: 2 copper layers, 304.8 x 119.1 mm, 378 parts, among them J1 USB_C_Receptacle_USB2.0_16P, J2 Conn_01x05, SW1 SW_Push, SW2 SW_Push, U1 RP2040, U2 XC6206PxxxMR, U3 W25Q128JVS, U85 74AHCT1G125, Y1 Crystal_GND24

Commit message: implement column traces of switch matrix
Routing:
- net COL11: track 0.00 -> 141.6 mm
- net COL9: track 0.00 -> 116.6 mm
- net COL10: track 0.00 -> 113.8 mm
- net COL1: track 0.00 -> 112.4 mm
- net COL2: track 0.00 -> 109.3 mm
- net COL13: track 0.00 -> 109.1 mm
- net COL5: track 0.00 -> 106.1 mm
- net COL0: track 0.00 -> 104.1 mm
- net COL14: track 0.00 -> 95.3 mm
- net COL6: track 0.00 -> 86.1 mm
- net COL4: track 0.00 -> 86.1 mm
- net COL3: track 0.00 -> 86.1 mm
- net COL8: track 0.00 -> 64.0 mm
- net COL12: track 0.00 -> 53.4 mm
